Commit message: Update

File: body.urdf (robot description, URDF)
Before this commit: robot robot, 6 links, 5 joints
Links:
- link 0: geometry collision box size=0.6942233505526942 0.4593124210216613 0.17989141607456896; visual box size=0.6942233505526942 0.4593124210216613 0.17989141607456896
- link 1: geometry collision box size=0.6942233505526942 0.4593124210216613 0.17989141607456896; visual box size=0.6942233505526942 0.4593124210216613 0.17989141607456896
- link 2: geometry collision box size=1.0687387083703608 0.7719698228034827 2.9469782028501994; visual box size=1.0687387083703608 0.7719698228034827 2.9469782028501994
- link 3: geometry collision box size=0.5343693541851804 0.38598491140174135 0.8473567978202724; visual box size=0.5343693541851804 0.38598491140174135 0.8473567978202724
- link 4: geometry collision box size=0.5343693541851804 0.38598491140174135 0.8473567978202724; visual box size=0.5343693541851804 0.38598491140174135 0.8473567978202724
- link Torso: geometry collision box size=1.3884467011053885 0.9186248420433226 0.44784004027931446; visual box size=1.3884467011053885 0.9186248420433226 0.44784004027931446
Joints:
- joint 2_3: origin xyz=0.5517726138139966 0.38359307300053636 -1.240196430718808 rpy=0 0 0 -> xyz=0.5343693541851804 0.38598491140174135 -1.4734891014250997 rpy=0 0 0
- joint 2_4: origin xyz=0.5517726138139966 -0.38359307300053636 -1.240196430718808 rpy=0 0 0 -> xyz=0.5343693541851804 -0.38598491140174135 -1.4734891014250997 rpy=0 0 0
- joint Torso_0: origin xyz=0 0 3.8553993457374274 rpy=0 0 0 -> xyz=0 0 3.776079979860343 rpy=0 0 0
- joint Torso_1: origin xyz=0 0 3.8553993457374274 rpy=0 0 0 -> xyz=0 0 3.776079979860343 rpy=0 0 0
- joint Torso_2: origin xyz=1.4692515581816106 0 4.0 rpy=0 0 0 -> xyz=0.6942233505526942 0 4.0 rpy=0 0 0
